File: $CurrentSinkOrSwim.sch (KiCad schematic (older format))
At the start: 4 parts, among them P101 ext pwr, P102 pwr select, P103 Input, P4 Gnd

Commit message: Changed footprints, changed layout
Connections:
- net Current Control/Current_Sink+: now also P103.2 (P2); no longer P103.1 (P1)
- net GND: now also P101.1 (P1), P103.1 (P1); no longer P101.2 (P2), P103.2 (P2)
- net at P102.1 (P1): now also P101.2 (P2); no longer P101.1 (P1)
Changed lines of the file:
@@
 F 4 "OSTTC022162" H 8300 1300 60  0001 C CNN "MPN"
 	1    8300 1300
-	1    0    0    -1
+	1    0    0    1
 $EndComp
 $Comp
@@
 F 4 "OSTTC022162" H 3000 850 60  0001 C CNN "MPN"
 	1    3000 850
-	-1   0    0    -1
+	-1   0    0    1
 $EndComp
 $Comp
