File: PowerRegulation.sch (KiCad schematic (older format))
At the start: 6 parts

Commit message: Initial Annotation
Parts:
- gave numbers to parts that had none: 6
Changed lines of the file:
@@
 $EndDescr
 $Comp
-L GND #PWR?
+L GND #PWR301
 U 1 1 54DAF107
 P 4800 3900
-F 0 "#PWR?" H 4800 3650 60  0001 C CNN
+F 0 "#PWR301" H 4800 3650 60  0001 C CNN
 F 1 "GND" H 4800 3750 60  0000 C CNN
 F 2 "" H 4800 3900 60  0000 C CNN
@@
 $EndComp
 $Comp
-L C C?
+L C C301
 U 1 1 54DAF10D
 P 4000 3300
-F 0 "C?" H 4050 3400 50  0000 L CNN
+F 0 "C301" H 4050 3400 50  0000 L CNN
 F 1 "C" H 4050 3200 50  0000 L CNN
 F 2 "" H 4038 3150 30  0000 C CNN
@@
 $EndComp
 $Comp
-L C C?
+L C C302
 U 1 1 54DAF114
 P 6200 3450
-F 0 "C?" H 6250 3550 50  0000 L CNN
+F 0 "C302" H 6250 3550 50  0000 L CNN
 F 1 "C" H 6250 3350 50  0000 L CNN
 F 2 "" H 6238 3300 30  0000 C CNN
@@
 	4000 3800 4000 3500
 $Comp
-L R R?
+L R R301
 U 1 1 54DAF11D
 P 4200 3200
-F 0 "R?" V 4280 3200 40  0000 C CNN
+F 0 "R301" V 4280 3200 40  0000 C CNN
 F 1 "0" V 4207 3201 40  0000 C CNN
 F 2 "" V 4130 3200 30  0000 C CNN
@@
 2.7V
 $Comp
-L LM2931D-R U?
+L LM2931D-R U301
 U 1 1 54DAF12F
 P 4750 3150
-F 0 "U?" H 5000 3000 60  0000 C CNN
+F 0 "U301" H 5000 3000 60  0000 C CNN
 F 1 "LM2931D-R" H 4750 3800 60  0000 C CNN
 F 2 "" H 4600 3150 60  0000 C CNN
@@
 Connection ~ 6200 2650
 $Comp
-L R R?
+L R R302
 U 1 1 54DAF13B
 P 5650 2900
-F 0 "R?" V 5730 2900 40  0000 C CNN
+F 0 "R302" V 5730 2900 40  0000 C CNN
 F 1 "27K" V 5657 2901 40  0000 C CNN
 F 2 "" V 5580 2900 30  0000 C CNN
@@
 $EndComp
 $Comp
-L R R?
+L R R303
 U 1 1 54DAF142
 P 5650 3550
-F 0 "R?" V 5730 3550 40  0000 C CNN
+F 0 "R303" V 5730 3550 40  0000 C CNN
 F 1 "21.6K" V 5657 3551 40  0000 C CNN
 F 2 "" V 5580 3550 30  0000 C CNN

Commit message: Preliminary association of components and placement into layout.
Parts:
- C301, C302, R301, R302, R303: footprint (none) -> SMD_Packages:SMD-0805
- U301: footprint (none) -> SMD_Packages:SOIC-8-N
Connections:
- wire segments 30 -> 20
Changed lines of the file:
@@
 $EndDescr
 $Comp
-L GND #PWR301
+L GND #PWR05
 U 1 1 54DAF107
 P 4800 3900
-F 0 "#PWR301" H 4800 3650 60  0001 C CNN
+F 0 "#PWR05" H 4800 3650 60  0001 C CNN
 F 1 "GND" H 4800 3750 60  0000 C CNN
 F 2 "" H 4800 3900 60  0000 C CNN
@@
 F 0 "C301" H 4050 3400 50  0000 L CNN
 F 1 "C" H 4050 3200 50  0000 L CNN
-F 2 "" H 4038 3150 30  0000 C CNN
+F 2 "SMD_Packages:SMD-0805" H 4038 3150 30  0001 C CNN
 F 3 "" H 4000 3300 60  0000 C CNN
 	1    4000 3300
@@
 F 0 "C302" H 6250 3550 50  0000 L CNN
 F 1 "C" H 6250 3350 50  0000 L CNN
-F 2 "" H 6238 3300 30  0000 C CNN
+F 2 "SMD_Packages:SMD-0805" H 6238 3300 30  0001 C CNN
 F 3 "" H 6200 3450 60  0000 C CNN
 	1    6200 3450
@@
 F 0 "R301" V 4280 3200 40  0000 C CNN
 F 1 "0" V 4207 3201 40  0000 C CNN
-F 2 "" V 4130 3200 30  0000 C CNN
+F 2 "SMD_Packages:SMD-0805" V 4130 3200 30  0001 C CNN
 F 3 "" H 4200 3200 30  0000 C CNN
 F 4 "Value" H 4200 3200 60  0001 C CNN "MPN"
@@
 $EndComp
 Wire Wire Line
-	4800 3450 4800 3800
+	4800 3450 4800 3900
 Wire Wire Line
-	4800 3800 4800 3850
-Wire Wire Line
-	4800 3850 4800 3900
-Wire Wire Line
-	4900 3800 4800 3800
-Wire Wire Line
-	4800 3800 4700 3800
-Wire Wire Line
-	4700 3800 4600 3800
-Wire Wire Line
-	4600 3800 4200 3800
-Wire Wire Line
-	4200 3800 4000 3800
+	4000 3800 4900 3800
 Connection ~ 4800 3800
 Wire Wire Line
@@
 F 0 "U301" H 5000 3000 60  0000 C CNN
 F 1 "LM2931D-R" H 4750 3800 60  0000 C CNN
-F 2 "" H 4600 3150 60  0000 C CNN
+F 2 "SMD_Packages:SOIC-8-N" H 4600 3150 60  0001 C CNN
 F 3 "" H 4600 3150 60  0000 C CNN
 	1    4750 3150
@@
 $EndComp
 Wire Wire Line
-	6850 2650 6200 2650
-Wire Wire Line
-	6200 2650 5200 2650
+	5200 2650 6850 2650
 Wire Wire Line
 	6200 2650 6200 3250
@@
 F 0 "R302" V 5730 2900 40  0000 C CNN
 F 1 "27K" V 5657 2901 40  0000 C CNN
-F 2 "" V 5580 2900 30  0000 C CNN
+F 2 "SMD_Packages:SMD-0805" V 5580 2900 30  0001 C CNN
 F 3 "" H 5650 2900 30  0000 C CNN
 F 4 "Value" H 5650 2900 60  0001 C CNN "MPN"
@@
 F 0 "R303" V 5730 3550 40  0000 C CNN
 F 1 "21.6K" V 5657 3551 40  0000 C CNN
-F 2 "" V 5580 3550 30  0000 C CNN
+F 2 "SMD_Packages:SMD-0805" V 5580 3550 30  0001 C CNN
 F 3 "" H 5650 3550 30  0000 C CNN
 	1    5650 3550
@@
 $EndComp
 Wire Wire Line
-	6200 3850 5650 3850
-Wire Wire Line
-	5650 3850 4800 3850
+	4800 3850 6200 3850
 Wire Wire Line
 	5650 3850 5650 3800
@@
 Connection ~ 5650 3850
 Wire Wire Line
-	5650 3150 5650 3250
-Wire Wire Line
-	5650 3250 5650 3300
+	5650 3150 5650 3300
 Wire Wire Line
 	5200 2850 5400 2850
@@
 	4900 3800 4900 3450
 Wire Wire Line
-	3750 2650 4000 2650
-Wire Wire Line
-	4000 2650 4300 2650
+	3750 2650 4300 2650
 Text GLabel 6850 2650 2    60   Input ~ 0
 2.7V

Commit message: Small changes after ERC check
Connections:
- wire segments 20 -> 21
Other:
- moved on the sheet: R302
Changed lines of the file:
@@
 	4000 3800 4900 3800
 Connection ~ 4800 3800
-Wire Wire Line
-	4200 2850 4200 3050
 Text Label 6200 4000 2    60   ~ 0
 2.7V
@@
 L R R302
 U 1 1 54DAF13B
-P 5650 2900
-F 0 "R302" V 5730 2900 40  0000 C CNN
-F 1 "27K" V 5657 2901 40  0000 C CNN
-F 2 "SMD_Packages:SMD-0805" V 5580 2900 30  0001 C CNN
-F 3 "" H 5650 2900 30  0000 C CNN
-F 4 "Value" H 5650 2900 60  0001 C CNN "MPN"
-	1    5650 2900
+P 5650 2950
+F 0 "R302" V 5730 2950 40  0000 C CNN
+F 1 "27K" V 5657 2951 40  0000 C CNN
+F 2 "SMD_Packages:SMD-0805" V 5580 2950 30  0001 C CNN
+F 3 "" H 5650 2950 30  0000 C CNN
+F 4 "Value" H 5650 2950 60  0001 C CNN "MPN"
+	1    5650 2950
 	-1   0    0    -1
 $EndComp
@@
 	6200 3850 6200 3650
 Connection ~ 5650 3850
-Wire Wire Line
-	5650 3150 5650 3300
 Wire Wire Line
 	5200 2850 5400 2850
@@
 Text HLabel 3750 2650 0    60   Input ~ 0
 Vin
+Wire Wire Line
+	4200 2850 4200 2950
+Wire Wire Line
+	5650 2700 5650 2650
+Connection ~ 5650 2650
+Wire Wire Line
+	5650 3200 5650 3300
 $EndSCHEMATC

Commit message: test netlist
Parts:
- renumbered C301 to C2, C302 to C3, R302 to R4, R301 to R5, R303 to R6, U301 to U2
Changed lines of the file:
@@
 $EndDescr
 $Comp
-L GND #PWR06
+L GND #PWR6
 U 1 1 54DAF107
 P 4800 3900
-F 0 "#PWR06" H 4800 3650 60  0001 C CNN
+F 0 "#PWR6" H 4800 3650 60  0001 C CNN
 F 1 "GND" H 4800 3750 60  0000 C CNN
 F 2 "" H 4800 3900 60  0000 C CNN
@@
 $EndComp
 $Comp
-L C C301
+L C C2
 U 1 1 54DAF10D
 P 4000 3300
-F 0 "C301" H 4050 3400 50  0000 L CNN
+F 0 "C2" H 4050 3400 50  0000 L CNN
 F 1 "C" H 4050 3200 50  0000 L CNN
 F 2 "SMD_Packages:SMD-0805" H 4038 3150 30  0001 C CNN
@@
 $EndComp
 $Comp
-L C C302
+L C C3
 U 1 1 54DAF114
 P 6200 3450
-F 0 "C302" H 6250 3550 50  0000 L CNN
+F 0 "C3" H 6250 3550 50  0000 L CNN
 F 1 "C" H 6250 3350 50  0000 L CNN
 F 2 "SMD_Packages:SMD-0805" H 6238 3300 30  0001 C CNN
@@
 	4000 3800 4000 3500
 $Comp
-L R R301
+L R R5
 U 1 1 54DAF11D
 P 4200 3200
-F 0 "R301" V 4280 3200 40  0000 C CNN
+F 0 "R5" V 4280 3200 40  0000 C CNN
 F 1 "0" V 4207 3201 40  0000 C CNN
 F 2 "SMD_Packages:SMD-0805" V 4130 3200 30  0001 C CNN
@@
 2.7V
 $Comp
-L LM2931D-R U301
+L LM2931D-R U2
 U 1 1 54DAF12F
 P 4750 3150
-F 0 "U301" H 5000 3000 60  0000 C CNN
+F 0 "U2" H 5000 3000 60  0000 C CNN
 F 1 "LM2931D-R" H 4750 3800 60  0000 C CNN
 F 2 "SMD_Packages:SOIC-8-N" H 4600 3150 60  0001 C CNN
@@
 Connection ~ 6200 2650
 $Comp
-L R R302
+L R R4
 U 1 1 54DAF13B
 P 5650 2950
-F 0 "R302" V 5730 2950 40  0000 C CNN
+F 0 "R4" V 5730 2950 40  0000 C CNN
 F 1 "27K" V 5657 2951 40  0000 C CNN
 F 2 "SMD_Packages:SMD-0805" V 5580 2950 30  0001 C CNN
@@
 $EndComp
 $Comp
-L R R303
+L R R6
 U 1 1 54DAF142
 P 5650 3550
-F 0 "R303" V 5730 3550 40  0000 C CNN
+F 0 "R6" V 5730 3550 40  0000 C CNN
 F 1 "21.6K" V 5657 3551 40  0000 C CNN
 F 2 "SMD_Packages:SMD-0805" V 5580 3550 30  0001 C CNN

Commit message: Routing done - Final
Just add artwork
Parts:
- renumbered C2 to C301, C3 to C302, R5 to R301, R4 to R302, R6 to R303, U2 to U301
Changed lines of the file:
@@
 $EndDescr
 $Comp
-L GND #PWR6
+L GND #PWR06
 U 1 1 54DAF107
 P 4800 3900
-F 0 "#PWR6" H 4800 3650 60  0001 C CNN
+F 0 "#PWR06" H 4800 3650 60  0001 C CNN
 F 1 "GND" H 4800 3750 60  0000 C CNN
 F 2 "" H 4800 3900 60  0000 C CNN
@@
 $EndComp
 $Comp
-L C C2
+L C C301
 U 1 1 54DAF10D
 P 4000 3300
-F 0 "C2" H 4050 3400 50  0000 L CNN
+F 0 "C301" H 4050 3400 50  0000 L CNN
 F 1 "C" H 4050 3200 50  0000 L CNN
 F 2 "SMD_Packages:SMD-0805" H 4038 3150 30  0001 C CNN
@@
 $EndComp
 $Comp
-L C C3
+L C C302
 U 1 1 54DAF114
 P 6200 3450
-F 0 "C3" H 6250 3550 50  0000 L CNN
+F 0 "C302" H 6250 3550 50  0000 L CNN
 F 1 "C" H 6250 3350 50  0000 L CNN
 F 2 "SMD_Packages:SMD-0805" H 6238 3300 30  0001 C CNN
@@
 	4000 3800 4000 3500
 $Comp
-L R R5
+L R R301
 U 1 1 54DAF11D
 P 4200 3200
-F 0 "R5" V 4280 3200 40  0000 C CNN
+F 0 "R301" V 4280 3200 40  0000 C CNN
 F 1 "0" V 4207 3201 40  0000 C CNN
 F 2 "SMD_Packages:SMD-0805" V 4130 3200 30  0001 C CNN
@@
 2.7V
 $Comp
-L LM2931D-R U2
+L LM2931D-R U301
 U 1 1 54DAF12F
 P 4750 3150
-F 0 "U2" H 5000 3000 60  0000 C CNN
+F 0 "U301" H 5000 3000 60  0000 C CNN
 F 1 "LM2931D-R" H 4750 3800 60  0000 C CNN
 F 2 "SMD_Packages:SOIC-8-N" H 4600 3150 60  0001 C CNN
@@
 Connection ~ 6200 2650
 $Comp
-L R R4
+L R R302
 U 1 1 54DAF13B
 P 5650 2950
-F 0 "R4" V 5730 2950 40  0000 C CNN
+F 0 "R302" V 5730 2950 40  0000 C CNN
 F 1 "27K" V 5657 2951 40  0000 C CNN
 F 2 "SMD_Packages:SMD-0805" V 5580 2950 30  0001 C CNN
@@
 $EndComp
 $Comp
-L R R6
+L R R303
 U 1 1 54DAF142
 P 5650 3550
-F 0 "R6" V 5730 3550 40  0000 C CNN
+F 0 "R303" V 5730 3550 40  0000 C CNN
 F 1 "21.6K" V 5657 3551 40  0000 C CNN
 F 2 "SMD_Packages:SMD-0805" V 5580 3550 30  0001 C CNN
