File: VoltageControl.sch (KiCad schematic (older format))
At the start: 8 parts, among them P5 V, U1 LMV358

Commit message: Routing done - Final
Just add artwork
Parts:
- renumbered C1 to C201, D1 to D201, P5 to P2, R1 to R201, R2 to R202, R3 to R203, RV1 to RV201, U1 to U201
Changed lines of the file:
@@
 $EndDescr
 $Comp
-L LMV358 U1
+L LMV358 U201
 U 1 1 54DB1D03
 P 5850 3050
-F 0 "U1" H 5800 3250 60  0000 L CNN
+F 0 "U201" H 5800 3250 60  0000 L CNN
 F 1 "LMV358" H 5800 2800 60  0000 L CNN
 F 2 "SMD_Packages:SOIC-8-N" H 5850 3050 60  0001 C CNN
@@
 $EndComp
 $Comp
-L R R1
+L R R201
 U 1 1 54DB1D0A
 P 4100 2650
-F 0 "R1" V 4180 2650 50  0000 C CNN
+F 0 "R201" V 4180 2650 50  0000 C CNN
 F 1 "28.7K" V 4107 2651 50  0000 C CNN
 F 2 "SMD_Packages:SMD-0805" V 4030 2650 30  0001 C CNN
@@
 $EndComp
 $Comp
-L GND #PWR5
+L GND #PWR04
 U 1 1 54DB1D11
 P 5750 3600
-F 0 "#PWR5" H 5750 3350 60  0001 C CNN
+F 0 "#PWR04" H 5750 3350 60  0001 C CNN
 F 1 "GND" H 5750 3450 60  0000 C CNN
 F 2 "" H 5750 3600 60  0000 C CNN
@@
 	3800 5550 9850 5550
 $Comp
-L POT RV1
+L POT RV201
 U 1 1 54DB1D22
 P 3800 3550
-F 0 "RV1" H 3800 3450 50  0000 C CNN
+F 0 "RV201" H 3800 3450 50  0000 C CNN
 F 1 "10K" H 3800 3550 50  0000 C CNN
 F 2 "Current:P090L-02F25BR10K" H 3800 3550 60  0001 C CNN
@@
 	5750 1950 5750 2650
 $Comp
-L GND #PWR4
+L GND #PWR05
 U 1 1 54DB1D2C
 P 5150 2650
-F 0 "#PWR4" H 5150 2400 60  0001 C CNN
+F 0 "#PWR05" H 5150 2400 60  0001 C CNN
 F 1 "GND" H 5150 2500 60  0000 C CNN
 F 2 "" H 5150 2650 60  0000 C CNN
@@
 $EndComp
 $Comp
-L C C1
+L C C201
 U 1 1 54DB1D32
 P 5150 2400
-F 0 "C1" H 5200 2500 50  0000 L CNN
+F 0 "C201" H 5200 2500 50  0000 L CNN
 F 1 "C" H 5200 2300 50  0000 L CNN
 F 2 "SMD_Packages:SMD-0805" H 5188 2250 30  0001 C CNN
@@
 	6350 3050 6550 3050
 $Comp
-L DIODE D1
+L DIODE D201
 U 1 1 54DB1E38
 P 6750 3050
-F 0 "D1" H 6750 3150 40  0000 C CNN
+F 0 "D201" H 6750 3150 40  0000 C CNN
 F 1 "DIODE" H 6750 2950 40  0000 C CNN
 F 2 "SMD_Packages:SOD-523" H 6750 3050 60  0001 C CNN
@@
 $EndComp
 $Comp
-L R R2
+L R R202
 U 1 1 54DB1EC2
 P 8700 3450
-F 0 "R2" V 8780 3450 50  0000 C CNN
+F 0 "R202" V 8780 3450 50  0000 C CNN
 F 1 "9K" V 8707 3451 50  0000 C CNN
 F 2 "SMD_Packages:SMD-0805" V 8630 3450 30  0001 C CNN
@@
 $EndComp
 $Comp
-L R R3
+L R R203
 U 1 1 54DB1F3A
 P 8700 4300
-F 0 "R3" V 8780 4300 50  0000 C CNN
+F 0 "R203" V 8780 4300 50  0000 C CNN
 F 1 "1K" V 8707 4301 50  0000 C CNN
 F 2 "SMD_Packages:SMD-0805" V 8630 4300 30  0001 C CNN
@@
 Connection ~ 4100 3550
 $Comp
-L CONN_01X01 P5
+L CONN_01X01 P2
 U 1 1 54F1F52A
 P 4400 3850
-F 0 "P5" H 4400 3950 50  0000 C CNN
+F 0 "P2" H 4400 3950 50  0000 C CNN
 F 1 "V" V 4500 3850 50  0000 C CNN
 F 2 "Pin_Headers:Pin_Header_Straight_1x01" H 4400 3850 60  0001 C CNN
